Commit message: wip: problem with gripper, moveit sim_time not complete

File: kortex_description/grippers/gen3_lite_2f/urdf/gen3_lite_2f.ros2_control.xacro (robot description, xacro)
@@ -32,5 +32,5 @@
                 <command_interface name="position" />
                 <state_interface name="position">
-                    <param name="initial_value">0.85</param>
+                    <param name="initial_value">0.75</param>
                 </state_interface>
                 <state_interface name="velocity"/>

File: kortex_description/grippers/gen3_lite_2f/urdf/gen3_lite_2f_macro.xacro (robot description, xacro)
@@ -124,5 +124,6 @@
       <child link="${prefix}right_finger_dist_link" />
       <axis xyz="0 0 1" />
-      <limit lower="-0.50" upper="0.21" effort="1000" velocity="1000" /> <!--limit lower="-1.03" upper="0.21" effort="1000" velocity="1000" /-->
+      <limit lower="-0.50" upper="0.21" effort="1000" velocity="1000" />
+      <!-- <limit lower="-1.03" upper="0.21" effort="1000" velocity="1000" /> -->
       <mimic joint="${prefix}right_finger_bottom_joint" multiplier="-0.676" offset="0.149" />
     </joint>
@@ -157,5 +158,5 @@
       <child link="${prefix}left_finger_prox_link" />
       <axis xyz="0 0 1" />
-      <limit lower="0.0" upper="0.85" effort="1000" velocity="1000" />
+      <limit lower="0.0" upper="0.96" effort="1000" velocity="1000" />
       <mimic joint="${prefix}right_finger_bottom_joint" multiplier="1.0" offset="0.0" />
     </joint>
@@ -190,5 +191,6 @@
       <child link="${prefix}left_finger_dist_link" />
       <axis xyz="0 0 -1" />
-      <limit lower="-0.50" upper="0.21" effort="1000" velocity="1000" /> <!--limit lower="-1.03" upper="0.21" effort="1000" velocity="1000" /-->
+      <limit lower="-0.50" upper="0.21" effort="1000" velocity="1000" />
+      <!-- <limit lower="-1.03" upper="0.21" effort="1000" velocity="1000" /> -->
       <mimic joint="${prefix}right_finger_bottom_joint" multiplier="-0.676" offset="0.149" />
     </joint>

Commit message: fix end effector tentative

File: kortex_description/grippers/gen3_lite_2f/urdf/gen3_lite_2f.ros2_control.xacro (robot description, xacro)
@@ -32,5 +32,5 @@
                 <command_interface name="position" />
                 <state_interface name="position">
-                    <param name="initial_value">0.85</param>
+                    <param name="initial_value">0.0</param>
                 </state_interface>
                 <state_interface name="velocity"/>
@@ -40,5 +40,5 @@
                 <joint name="${prefix}right_finger_tip_joint">
                     <param name="mimic">${prefix}right_finger_bottom_joint</param>
-                    <param name="multiplier">-1</param>
+                    <param name="multiplier">1</param>
                     <xacro:unless value="${sim_ignition}">
                         <command_interface name="position"/>
@@ -58,5 +58,5 @@
                 <joint name="${prefix}left_finger_tip_joint">
                     <param name="mimic">${prefix}right_finger_bottom_joint</param>
-                    <param name="multiplier">-1</param>
+                    <param name="multiplier">1</param>
                     <xacro:unless value="${sim_ignition}">
                         <command_interface name="position"/>

File: kortex_description/grippers/gen3_lite_2f/urdf/gen3_lite_2f_macro.xacro (robot description, xacro)
@@ -123,5 +123,5 @@
       <parent link="${prefix}right_finger_prox_link" />
       <child link="${prefix}right_finger_dist_link" />
-      <axis xyz="0 0 1" />
+      <axis xyz="0 0 -1" />
       <limit lower="-0.50" upper="0.21" effort="1000" velocity="1000" />
       <!-- <limit lower="-1.03" upper="0.21" effort="1000" velocity="1000" /> -->
@@ -190,5 +190,5 @@
       <parent link="${prefix}left_finger_prox_link" />
       <child link="${prefix}left_finger_dist_link" />
-      <axis xyz="0 0 -1" />
+      <axis xyz="0 0 1" />
       <limit lower="-0.50" upper="0.21" effort="1000" velocity="1000" />
       <!-- <limit lower="-1.03" upper="0.21" effort="1000" velocity="1000" /> -->

File: kortex_description/grippers/gen3_lite_2f/urdf/gen3_lite_2f_transmission_macro.xacro (robot description, xacro)
@@ -16,26 +16,26 @@
                 <joint>${prefix}right_finger_bottom_joint</joint>
                 <mimicJoint>${prefix}right_finger_tip_joint</mimicJoint>
-                <multiplier>-0.676</multiplier>
+                <multiplier>0.676</multiplier>
                 <offset>0.149</offset>
                 <maxEffort>5.0</maxEffort>
-                <hasPID></hasPID>
+                <sensitiveness>0.001</sensitiveness>
             </plugin>
             <plugin filename="libroboticsgroup_gazebo_mimic_joint_plugin.so" name="mimic_gen3_lite_2f_2">
                 <joint>${prefix}right_finger_bottom_joint</joint>
                 <mimicJoint>${prefix}left_finger_bottom_joint</mimicJoint>
-                <multiplier>-1.0</multiplier>
+                <multiplier>1.0</multiplier>
                 <offset>0.0</offset>
                 <maxEffort>5.0</maxEffort>
-                <hasPID></hasPID>
+                <sensitiveness>0.001</sensitiveness>
             </plugin>
             <plugin filename="libroboticsgroup_gazebo_mimic_joint_plugin.so" name="mimic_gen3_lite_2f_3">
                 <joint>${prefix}right_finger_bottom_joint</joint>
                 <mimicJoint>${prefix}left_finger_tip_joint</mimicJoint>
-                <multiplier>-0.676</multiplier>
+                <multiplier>0.676</multiplier>
                 <offset>0.149</offset>
                 <maxEffort>5.0</maxEffort>
-                <hasPID></hasPID>
+                <sensitiveness>0.001</sensitiveness>
             </plugin>
-            <plugin name="gazebo_grasp_fix" filename="libgazebo_grasp_fix.so">
+            <!-- <plugin name="gazebo_grasp_fix" filename="libgazebo_grasp_fix.so">
                 <arm>
                     <arm_name>my_gen3_lite_gripper</arm_name>
@@ -51,5 +51,5 @@
                 <disable_collisions_on_attach>false</disable_collisions_on_attach>
                 <contact_topic>__default_topic__</contact_topic>
-            </plugin>
+            </plugin> -->
         </gazebo>
     </xacro:macro>

Commit message: workaround for not implemented gripper interface

File: kortex_description/grippers/gen3_lite_2f/urdf/gen3_lite_2f.ros2_control.xacro (robot description, xacro)
@@ -1,5 +1,6 @@
 <?xml version="1.0"?>
 <robot xmlns:xacro="http://www.ros.org/wiki/xacro">
-    <xacro:macro name="gripper_ros2_control" params="
+    <xacro:macro name="gripper_ros2_control"
+        params="
         prefix
         use_fake_hardware:=false
@@ -10,61 +11,65 @@
         isaac_joint_states:=/isaac_joint_states
         use_internal_bus_gripper_comm:=false">
-        <ros2_control name="GripperHardwareInterface" type="system">
-            <hardware>
-                <xacro:if value="${sim_isaac}">
-                    <plugin>topic_based_ros2_control/TopicBasedSystem</plugin>
-                    <param name="joint_commands_topic">${isaac_joint_commands}</param>
-                    <param name="joint_states_topic">${isaac_joint_states}</param>
-                    <param name="trigger_joint_command_threshold">0.02</param>
+        <xacro:if value="${use_fake_hardware or sim_isaac or sim_ignition}">
+            <ros2_control name="GripperHardwareInterface" type="system">
+                <hardware>
+                    <xacro:if value="${sim_isaac}">
+                        <plugin>topic_based_ros2_control/TopicBasedSystem</plugin>
+                        <param name="joint_commands_topic">${isaac_joint_commands}</param>
+                        <param name="joint_states_topic">${isaac_joint_states}</param>
+                        <param name="trigger_joint_command_threshold">0.02</param>
+                    </xacro:if>
+                    <xacro:if value="${sim_ignition}">
+                        <plugin>ign_ros2_control/IgnitionSystem</plugin>
+                    </xacro:if>
+                    <xacro:if value="${use_fake_hardware}">
+                        <plugin>mock_components/GenericSystem</plugin>
+                        <param name="fake_sensor_commands">${fake_sensor_commands}</param>
+                        <param name="state_following_offset">0.0</param>
+                    </xacro:if>
+                </hardware>
+                <!-- Joint interfaces -->
+                <!-- With Ignition or Hardware, they handle mimic joints, so we only need this
+                command
+            interface activated -->
+                <joint name="${prefix}right_finger_bottom_joint">
+                    <command_interface name="position" />
+                    <state_interface name="position">
+                        <param name="initial_value">0.85</param>
+                    </state_interface>
+                    <state_interface name="velocity" />
+                </joint>
+                <!-- When simulating we need to include the rest of the gripper joints -->
+                <xacro:if value="${use_fake_hardware or sim_isaac or sim_ignition}">
+                    <joint name="${prefix}right_finger_tip_joint">
+                        <param name="mimic">${prefix}right_finger_bottom_joint</param>
+                        <param name="multiplier">-1</param>
+                        <xacro:unless value="${sim_ignition}">
+                            <command_interface name="position" />
+                            <state_interface name="position" />
+                            <state_interface name="velocity" />
+                        </xacro:unless>
+                    </joint>
+                    <joint name="${prefix}left_finger_bottom_joint">
+                        <param name="mimic">${prefix}right_finger_bottom_joint</param>
+                        <param name="multiplier">1</param>
+                        <xacro:unless value="${sim_ignition}">
+                            <command_interface name="position" />
+                            <state_interface name="position" />
+                            <state_interface name="velocity" />
+                        </xacro:unless>
+                    </joint>
+                    <joint name="${prefix}left_finger_tip_joint">
+                        <param name="mimic">${prefix}right_finger_bottom_joint</param>
+                        <param name="multiplier">-1</param>
+                        <xacro:unless value="${sim_ignition}">
+                            <command_interface name="position" />
+                            <state_interface name="position" />
+                            <state_interface name="velocity" />
+                        </xacro:unless>
+                    </joint>
                 </xacro:if>
-                <xacro:if value="${sim_ignition}">
-                    <plugin>ign_ros2_control/IgnitionSystem</plugin>
-                </xacro:if>
-                <xacro:if value="${use_fake_hardware}">
-                    <plugin>mock_components/GenericSystem</plugin>
-                    <param name="fake_sensor_commands">${fake_sensor_commands}</param>
-                    <param name="state_following_offset">0.0</param>
-                </xacro:if>
-            </hardware>
-            <!-- Joint interfaces -->
-            <!-- With Ignition or Hardware, they handle mimic joints, so we only need this command interface activated -->
-            <joint name="${prefix}right_finger_bottom_joint">
-                <command_interface name="position" />
-                <state_interface name="position">
-                    <param name="initial_value">0.85</param>
-                </state_interface>
-                <state_interface name="velocity"/>
-            </joint>
-            <!-- When simulating we need to include the rest of the gripper joints -->
-            <xacro:if value="${use_fake_hardware or sim_isaac or sim_ignition}">
-                <joint name="${prefix}right_finger_tip_joint">
-                    <param name="mimic">${prefix}right_finger_bottom_joint</param>
-                    <param name="multiplier">-1</param>
-                    <xacro:unless value="${sim_ignition}">
-                        <command_interface name="position"/>
-                        <state_interface name="position"/>
-                        <state_interface name="velocity"/>
-                    </xacro:unless>
-                </joint>
-                <joint name="${prefix}left_finger_bottom_joint">
-                    <param name="mimic">${prefix}right_finger_bottom_joint</param>
-                    <param name="multiplier">1</param>
-                    <xacro:unless value="${sim_ignition}">
-                        <command_interface name="position"/>
-                        <state_interface name="position"/>
-                        <state_interface name="velocity"/>
-                    </xacro:unless>
-                </joint>
-                <joint name="${prefix}left_finger_tip_joint">
-                    <param name="mimic">${prefix}right_finger_bottom_joint</param>
-                    <param name="multiplier">-1</param>
-                    <xacro:unless value="${sim_ignition}">
-                        <command_interface name="position"/>
-                        <state_interface name="position"/>
-                        <state_interface name="velocity"/>
-                    </xacro:unless>
-                </joint>
-            </xacro:if>
-        </ros2_control>
+            </ros2_control>
+        </xacro:if>
     </xacro:macro>
 </robot>
